File: Badge_hw/Badge.kicad_pcb (KiCad board)
At the start: 2 copper layers, 35.5 x 27 mm, 42 parts, among them Q1 IRLML9303, SW1 BUTTON, U1 Round2.2

Commit message: Badge2 pcb routed
Parts:
- removed C12, C13: 20pF, Capacitors:CAP_0603
- removed R6: 200R, Resistors:RES_0603
- removed XTAL1: 12MHz, Quartz:0503x4-4
- added B1: BAT, Installation:BATTERY_CH7410, B.Cu at (147.2, 80.2)
- added C19: 4.7u, Capacitors:CAP_0603, F.Cu at (164.0, 79.1)
- added D2: BAT54WS, Diodes:SOD323, F.Cu at (164.0, 83.2)
- added Q2: MMBT2222, SOT:SOT23-3, F.Cu at (161.0, 83.6)
- added R10: 10k, Resistors:RES_0603, F.Cu at (153.0, 78.2)
- added R11: 1k, Resistors:RES_0603, F.Cu at (161.2, 79.8)
- added SW2: IT-1198E, BtnsSwitches:BTN_IT1198, B.Cu at (165.6, 88.7)
- added SW3: IT-1198E, BtnsSwitches:BTN_IT1198, F.Cu at (165.6, 88.7)
- added XL6: CONN_2, Connectors:PLS-2, F.Cu at (166.3, 81.4)
- SW1: value BUTTON -> IT-1187; moved to B.Cu
- XL3: moved to B.Cu
- moved XL1 79.0 mm to (143.4, 59.8)
- moved R5 71.8 mm to (138.5, 69.6), turned to 90 degrees
- moved XL3 71.2 mm to (131.2, 67.0), turned to 241 degrees
- moved C18 69.9 mm to (134.9, 69.6), turned to 90 degrees
- moved R9 69.2 mm to (133.1, 69.6), turned to 90 degrees
- moved C16 68.7 mm to (140.4, 63.6), turned to 35 degrees
- moved DD2 66.7 mm to (143.1, 69.0)
- moved R7 63.8 mm to (156.2, 65.4), turned to 90 degrees
- moved XL4 63.7 mm to (135.4, 63.7), turned to 33 degrees
- moved C11 62.6 mm to (158.2, 65.4), turned to 90 degrees
- moved R8 62.2 mm to (147.0, 67.0), turned to 90 degrees
- moved C3 61.7 mm to (142.6, 76.6)
- moved C4 60.4 mm to (138.2, 86.0), turned to 90 degrees
- moved SW1 60.1 mm to (154.6, 65.8), turned to 90 degrees
- moved R4 58.8 mm to (161.8, 69.6), turned to 90 degrees
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Connections:
- net Net-(DD1-Pad11) renamed /BatMeas
- DD1 pad 2: Net-(DD1-Pad2) -> /Vibro
- DD1 pad 3: Net-(DD1-Pad3) -> /Charge
- DD1 pad 38: /Charge -> Net-(DD1-Pad38)
- DD1 pad 4: Net-(DD1-Pad4) -> (no net)
- DD1 pad 5: Net-(C13-Pad1) -> Net-(DD1-Pad5)
- DD1 pad 6: Net-(DD1-Pad6) -> (no net)
- R5 pad 2: Net-(DD1-Pad2) -> Net-(DD1-Pad5)
Routing:
- net GND: track 0.00 -> 299.9 mm, vias 0 -> 44
- net +3.3V: track 0.00 -> 152.2 mm, vias 0 -> 9
- net +5V: track 0.00 -> 46.3 mm, vias 0 -> 5
- net Net-(DD1-Pad10): track 0.00 -> 39.1 mm, vias 0 -> 5
- net /SWCLK: track 0.00 -> 36.1 mm, vias 0 -> 1
- net /SHLD: track 0.00 -> 34.4 mm, vias 0 -> 4
- net /SWDIO: track 0.00 -> 32.9 mm, vias 0 -> 1
- net Net-(DD1-Pad5): track 0.00 -> 22.5 mm, vias 0 -> 2
- net /LCD_IMO: track 0.00 -> 22.2 mm, vias 0 -> 1
- net /IR_RX: track 0.00 -> 21.5 mm, vias 0 -> 1
- net /LED_C2: track 0.00 -> 21.3 mm, vias 0 -> 2
- net /BatMeas: track 0.00 -> 19.6 mm, vias 0 -> 2
- net /Charge: track 0.00 -> 19.3 mm, vias 0 -> 2
- net /LED_C1: track 0.00 -> 19.2 mm, vias 0 -> 2
- net /LCD_RS: track 0.00 -> 19.1 mm, vias 0 -> 1
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- added copper zone on B.Cu, net GND
- added copper zone on F.Cu, net GND
Other:
- board size 35.5 x 27 mm -> 41.6 x 38.4 mm
- net class Default: trace_width 0.25 -> 0.2; via_dia 0.6 -> 0.7; via_drill 0.4 -> 0.3
- net class Wide added: clearance 0.2, trace_width 0.5, via_dia 0.9, via_drill 0.4
- rule pad_to_mask_clearance: 0.2 -> 0.1

Commit message: + Badge3 PCB completed
Parts:
- removed C16: 0.1u, Capacitors:CAP_0603
- removed C19: 4.7u, Capacitors:CAP_0603
- removed D2: BAT54WS, Diodes:SOD323
- removed SW3: IT-1198E, BtnsSwitches:BTN_IT1198
- removed XL5, XL6: CONN_2, Connectors:PLS-2
- added C12: 0.1u, Capacitors:CAP_0603, F.Cu at (162.4, 90.9)
- added F1: Fuse0R, Resistors:RES_0603_FUSE, B.Cu at (165.9, 72.9)
- added F2: Fuse0R, Resistors:RES_0603_FUSE, F.Cu at (148.3, 67.4)
- added R6: 100k, Resistors:RES_0603, F.Cu at (151.3, 66.6)
- B1: footprint Installation:BATTERY_CH7410 -> Installation:EEMB603030
- C7: value 0.1u -> 10n
- C9: value 0.1u -> 1u
- DD2: footprint SO_DIL_TSSOP:SO8 -> SO_DIL_TSSOP:SO8_208MIL
- Q2: value MMBT2222 -> IRLML9303
- R11: value 1k -> 100R
- R7: value 2k -> 4k7
- R8: value 51k -> 100k
- SW1: value IT-1187 -> SWITCH; footprint BtnsSwitches:BTN_4x4_SMD -> BtnsSwitches:SW_SS-1P2T
- SW2: moved to F.Cu
- moved XL4 40.5 mm to (164.7, 91.6), turned to 90 degrees
- moved Q2 21.2 mm to (148.4, 66.6), turned to 270 degrees
- moved C9 13.1 mm to (148.7, 69.9)
- moved SW1 12.6 mm to (164.1, 74.1), turned to 270 degrees
- moved C10 10.4 mm to (158.4, 81.0), turned to 90 degrees
- moved R4 10.2 mm to (155.0, 77.2), turned to 180 degrees
- moved DA1 10.1 mm to (160.9, 80.9), turned to 270 degrees
- moved C2 8.50 mm to (153.9, 81.9), turned to 270 degrees
- moved R11 7.60 mm to (162.4, 87.3), turned to 90 degrees
- moved XL1 7.37 mm to (150.8, 59.8), turned to 180 degrees
- moved SW2 7.36 mm to (166.5, 81.4), turned to 90 degrees
- moved C5 5.99 mm to (160.6, 78.1), turned to 180 degrees
- moved R8 3.11 mm to (146.8, 63.9)
- moved D1 2.91 mm to (157.5, 73.1)
- moved Q1 2.91 mm to (160.4, 73.2)
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Connections:
- B1 pad A: +3.3V -> /BAT
- C1 pad 1: +3.3V -> /LCD_PWR
- C15 pad 1: +3.3V -> /MEM_PWR
- C9 pad 1: +3.3V -> /MEM_PWR
- DD1 pad 10: Net-(DD1-Pad10) -> /Btn
- DD1 pad 2: /Vibro -> /MEM_PWR_CTRL
- DD1 pad 26: /LCD_IMO -> /LCD_PWR
- DD1 pad 4: (no net) -> /IR_PWR
- DD2 pad 8: +3.3V -> /MEM_PWR
- Q2 pad 1: Net-(Q2-Pad1) -> /MEM_PWR_CTRL
- Q2 pad 2: GND -> +3.3V
- Q2 pad 3: /VibroOut -> /MEM_PWR
- R11 pad 1: /Vibro -> Net-(C12-Pad2)
- R11 pad 2: Net-(Q2-Pad1) -> /IR_PWR
- R8 pad 1: +3.3V -> /MEM_PWR
- SW1 pad 1: Net-(DD1-Pad10) -> /BAT
- SW1 pad 2: +3.3V -> +BATT
- SW2 pad 2: Net-(DD1-Pad10) -> /Btn
- U1 pad 2: +3.3V -> /LCD_PWR
- U1 pad 26: /LCD_IMO -> (no net)
- U1 pad 3: +3.3V -> /LCD_PWR
- XL4 pad 3: +3.3V -> Net-(C12-Pad2)
Routing:
- net +3.3V: track 152.2 -> 101.5 mm, vias 9 -> 6
- net Net-(DD1-Pad10): track 39.1 -> 0.00 mm, vias 5 -> 0
- net GND: track 299.9 -> 272.6 mm, vias 44 -> 52
- net /MEM_PWR_CTRL: track 0.00 -> 22.3 mm
- net /LCD_IMO: track 22.2 -> 0.00 mm, vias 1 -> 0
- net /LCD_PWR: track 0.00 -> 18.1 mm, vias 0 -> 3
- net /Btn: track 0.00 -> 17.1 mm, vias 0 -> 2
- net /BAT: track 0.00 -> 14.2 mm
- net /IR_PWR: track 0.00 -> 13.5 mm, vias 0 -> 2
- net /Vibro: track 13.2 -> 0.00 mm
- net /BatMeas: track 19.6 -> 7.05 mm, vias 2 -> 0
- net +BATT: track 11.2 -> 21.8 mm, vias 0 -> 1
- net /MEM_PWR: track 0.00 -> 9.18 mm
- net /VibroOut: track 5.45 -> 0.00 mm
- net /IR_RX: track 21.5 -> 26.7 mm
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Other:
- board text added: "Badge3"
- board text added: "Charger"
- board text added: "IR"
- board text added: "MEM"
- board text added: "USB"
